Commit message: new Robot Dimensions

File: catkin_ws/src/my_robot/urdf/twoWheelRobot.xacro (robot description, xacro)
@@ -1,5 +1,5 @@
 <?xml version='1.0'?>
 <robot name="my_robot" xmlns:xacro="http://www.ros.org/wiki/xacro">
-     <xacro:include filename="$(find my_robot)/urdf/my_robot.gazebo" />
+     <xacro:include filename="$(find my_robot)/urdf/twoWheelRobot.gazebo" />
     <link name="robot_footprint"></link>
     <joint name="robot_footprint_joint" type="fixed">
@@ -9,7 +9,8 @@
     </joint>
     <link name='chassis'>
+        <pose> 0 0 0.1 0 0 0 </pose>
         <visual name="chassis_visual">
             <geometry>
-                <box size='0.6 0.3 0.2' />
+                <box size='0.6 0.45 0.2' />
             </geometry>
             <origin xyz="0 0 0" rpy="0 0 0" />
@@ -25,7 +26,7 @@
             <origin xyz="0.0 0 0" rpy=" 0 0 0" />
             <inertia
-                ixx="0.21666666666666667" ixy="0" ixz="0"
+                ixx="0.4041666666666673" ixy="0" ixz="0"
                 iyy="0.6666666666666667" iyz="0"
-                izz="0.75"
+                izz="0.9375"
             />
         </inertial>
@@ -137,5 +138,5 @@
     </link>
     <joint type="fixed" name="camera_joint">
-        <origin xyz="0.2 0 0" rpy="0 0 0" />
+        <origin xyz="0.3 0 0" rpy="0 0 0" />
         <child link="camera" />
         <parent link="chassis" />
@@ -162,5 +163,5 @@
     </link>
     <joint type="fixed" name="hokuyo_joint">
-        <origin xyz="0.15 0 0.1" rpy="0 0 0" />
+        <origin xyz="0.2 0 0.1" rpy="0 0 0" />
         <child link="hokuyo" />
         <parent link="chassis" />
