Commit message: Update the origin of camera joint

File: catkin_ws/src/my_robot/urdf/my_robot.xacro (robot description, xacro)
@@ -138,5 +138,5 @@
     </link>
      <joint type="fixed" name="camera_joint">
-        <origin xyz="0.2, 0, 0" rpy="0 0 0"/>
+        <origin xyz="0.2 0 0" rpy="0 0 0"/>
         <child link="camera"/>
         <parent link="chassis"/>

Commit message: Update new world added

File: catkin_ws/src/my_robot/urdf/my_robot.xacro (robot description, xacro)
@@ -178,5 +178,5 @@
     </gazebo>
     <gazebo reference="camera">
-        <material>Gazebo/camera</material>
+        <material>Gazebo/Red</material>
     </gazebo>
 </robot>

Commit message: Finalized the Robot

File: catkin_ws/src/my_robot/urdf/my_robot.xacro (robot description, xacro)
@@ -1,5 +1,5 @@
 <?xml version='1.0'?>
 <robot name="my_robot" xmlns:xacro="http://www.ros.org/wiki/xacro">
-    <xacro:include filename="$(find my_robot)/urdf/my_robot.gazebo" />
+     <xacro:include filename="$(find my_robot)/urdf/twoWheelRobot.gazebo" />
     <link name="robot_footprint"></link>
     <joint name="robot_footprint_joint" type="fixed">
@@ -9,71 +9,71 @@
     </joint>
     <link name='chassis'>
-        <pose>0 0 0.1 0 0 0</pose>
+        <pose> 0 0 0.1 0 0 0 </pose>
+        <visual name="chassis_visual">
+            <geometry>
+                <box size='0.6 0.45 0.2' />
+            </geometry>
+            <origin xyz="0 0 0" rpy="0 0 0" />
+        </visual>
+        <collision name="chassis_collision">
+            <geometry>
+                <box size='0.6 0.3 0.2' />
+            </geometry>
+            <origin xyz="0 0 0" rpy="0 0 0" />
+        </collision>
         <inertial>
-            <mass value="15.0"/>
-            <origin xyz="0.0 0 0" rpy=" 0 0 0"/>
+            <mass value="20.0" />
+            <origin xyz="0.0 0 0" rpy=" 0 0 0" />
             <inertia
-                ixx="0.1" ixy="0" ixz="0"
-                iyy="0.1" iyz="0"
-                izz="0.1"
+                ixx="0.4041666666666673" ixy="0" ixz="0"
+                iyy="0.6666666666666667" iyz="0"
+                izz="0.9375"
             />
         </inertial>
-        <collision name='collision'>
-            <origin xyz="0 0 0" rpy=" 0 0 0"/>
+        <collision name='back_caster_collision'>
+            <origin xyz="-0.15 0 -0.05" rpy=" 0 0 0" />
             <geometry>
-            <box size=".4 .2 .1"/>
-            </geometry>
-        </collision>
-        <visual name='chassis_visual'>
-            <origin xyz="0 0 0" rpy=" 0 0 0"/>
-            <geometry>
-            <box size=".4 .2 .1"/>
-            </geometry>
-        </visual>
-        <collision name='back_caster_collision'>
-            <origin xyz="-0.15 0 -0.05" rpy=" 0 0 0"/>
-            <geometry>
-            <sphere radius="0.0499"/>
+                <sphere radius="0.0499" />
             </geometry>
         </collision>
         <visual name='back_caster_visual'>
-            <origin xyz="-0.15 0 -0.05" rpy=" 0 0 0"/>
+            <origin xyz="-0.15 0 -0.05" rpy=" 0 0 0" />
             <geometry>
-            <sphere radius="0.05"/>
+                <sphere radius="0.05" />
             </geometry>
         </visual>
         <collision name='front_caster_collision'>
-            <origin xyz="0.15 0 -0.05" rpy=" 0 0 0"/>
+            <origin xyz="0.15 0 -0.05" rpy=" 0 0 0" />
             <geometry>
-            <sphere radius="0.0499"/>
+                <sphere radius="0.0499" />
             </geometry>
         </collision>
         <visual name='front_caster_visual'>
-            <origin xyz="0.15 0 -0.05" rpy=" 0 0 0"/>
+            <origin xyz="0.15 0 -0.05" rpy=" 0 0 0" />
             <geometry>
-            <sphere radius="0.05"/>
+                <sphere radius="0.05" />
             </geometry>
         </visual>
     </link>
-    <link name='left_wheel'>
+    <link name="left_wheel">
         <collision name='left_wheel_collision'>
-            <origin xyz="0 0 0" rpy=" 0 1.5707 1.5707"/>
+            <origin xyz="0 0 0" rpy=" 0 1.5707 1.5707" />
             <geometry>
-                <cylinder radius="0.1" length="0.05"/>
+                <cylinder radius="0.15" length="0.05" />
             </geometry>
         </collision>
         <visual name='left_wheel_visual'>
-            <origin xyz="0 0 0" rpy=" 0 1.5707 1.5707"/>
+            <origin xyz="0 0 0" rpy=" 0 1.5707 1.5707" />
             <geometry>
-                <cylinder radius="0.1" length="0.05"/>
+                <cylinder radius="0.15" length="0.05" />
             </geometry>
         </visual>
         <inertial>
-            <mass value="5.0"/>
-            <origin xyz="0.0 0 0" rpy=" 0 1.5707 1.5707"/>
+            <mass value="5.0" />
+            <origin xyz="0.0 0 0" rpy=" 0 1.5707 1.5707" />
             <inertia
-                ixx="0.1" ixy="0" ixz="0"
-                iyy="0.1" iyz="0"
-                izz="0.1"
+                ixx="0.02916666666666667" ixy="0" ixz="0"
+                iyy="0.02916666666666667" iyz="0"
+                izz="0.056249999999999994"
             />
         </inertial>
@@ -81,40 +81,40 @@
     <link name='right_wheel'>
         <collision name='right_wheel_collision'>
-            <origin xyz="0 0 0" rpy=" 0 1.5707 1.5707"/>
+            <origin xyz="0 0 0" rpy=" 0 1.5707 1.5707" />
             <geometry>
-                <cylinder radius="0.1" length="0.05"/>
+                <cylinder radius="0.15" length="0.05" />
             </geometry>
         </collision>
         <visual name='right_wheel_visual'>
-            <origin xyz="0 0 0" rpy=" 0 1.5707 1.5707"/>
+            <origin xyz="0 0 0" rpy=" 0 1.5707 1.5707" />
             <geometry>
-                <cylinder radius="0.1" length="0.05"/>
+                <cylinder radius="0.15" length="0.05" />
             </geometry>
         </visual>
         <inertial>
-            <mass value="5.0"/>
-            <origin xyz="0.0 0 0" rpy=" 0 1.5707 1.5707"/>
+            <mass value="5.0" />
+            <origin xyz="0.0 0 0" rpy=" 0 1.5707 1.5707" />
             <inertia
-                ixx="0.1" ixy="0" ixz="0"
-                iyy="0.1" iyz="0"
-                izz="0.1"
+                ixx="0.02916666666666667" ixy="0" ixz="0"
+                iyy="0.02916666666666667" iyz="0"
+                izz="0.056249999999999994"
             />
         </inertial>
     </link>
     <joint type="continuous" name="left_wheel_hinge">
-        <origin xyz="0 0.15 0" rpy="0 0 0"/>
-        <child link="left_wheel"/>
-        <parent link="chassis"/>
-        <axis xyz="0 1 0" rpy="0 0 0"/>
-        <limit effort="10000" velocity="1000"/>
-        <dynamics damping="1.0" friction="1.0"/>
+        <origin xyz="0 0.25 0" rpy="0 0 0" />
+        <child link="left_wheel" />
+        <parent link="chassis" />
+        <axis xyz="0 1 0" rpy="0 0 0" />
+        <limit effort="10000" velocity="1000" />
+        <dynamics damping="1.0" friction="1.0" />
     </joint>
     <joint type="continuous" name="right_wheel_hinge">
-        <origin xyz="0 -0.15 0" rpy="0 0 0"/>
-        <child link="right_wheel"/>
-        <parent link="chassis"/>
-        <axis xyz="0 1 0" rpy="0 0 0"/>
-        <limit effort="10000" velocity="1000"/>
-        <dynamics damping="1.0" friction="1.0"/>
+        <origin xyz="0 -0.25 0" rpy="0 0 0" />
+        <child link="right_wheel" />
+        <parent link="chassis" />
+        <axis xyz="0 1 0" rpy="0 0 0" />
+        <limit effort="10000" velocity="1000" />
+        <dynamics damping="1.0" friction="1.0" />
     </joint>
     <link name="camera">
@@ -122,5 +122,5 @@
             <origin xyz="0 0 0" rpy=" 0 0 0" />
             <geometry>
-                <box size= "0.05 0.05 0.05"/>
+                <box size="0.05 0.05 0.05" />
             </geometry>
         </collision>
@@ -128,18 +128,18 @@
             <origin xyz="0 0 0" rpy=" 0 0 0" />
             <geometry>
-                <box size= "0.05 0.05 0.05"/>
+                <box size="0.05 0.05 0.05" />
             </geometry>
         </visual>
         <inertial>
-            <mass value="0.1"/>
-            <origin xyz="0 0 0" rpy=" 0 0 0"/>
+            <mass value="0.1" />
+            <origin xyz="0 0 0" rpy=" 0 0 0" />
             <inertia ixx="1e-6" ixy="0" ixz="0" iyy="1e-6" iyz="0" izz="1e-6" />
         </inertial>
     </link>
-     <joint type="fixed" name="camera_joint">
-        <origin xyz="0.2 0 0" rpy="0 0 0"/>
-        <child link="camera"/>
-        <parent link="chassis"/>
-        <axis xyz="0 1 0" rpy="0 0 0"/>
+    <joint type="fixed" name="camera_joint">
+        <origin xyz="0.3 0 0" rpy="0 0 0" />
+        <child link="camera" />
+        <parent link="chassis" />
+        <axis xyz="0 1 0" rpy="0 0 0" />
     </joint>
     <link name="hokuyo">
@@ -147,5 +147,5 @@
             <origin xyz="0 0 0" rpy=" 0 0 0" />
             <geometry>
-                <box size= "0.1 0.1 0.1"/>
+                <box size="0.1 0.1 0.1" />
             </geometry>
         </collision>
@@ -153,30 +153,30 @@
             <origin xyz="0 0 0" rpy=" 0 0 0" />
             <geometry>
-                <mesh filename = "package://my_robot/meshes/hokuyo.dae"/>
+                <mesh filename="package://my_robot/meshes/hokuyo.dae" />
             </geometry>
         </visual>
         <inertial>
-            <mass value="1e-5"/>
-            <origin xyz="0 0 0" rpy=" 0 0 0"/>
-            <inertia ixx="1e-6" ixy="0" ixz="0" iyy="1e-6" iyz="0" izz="1e-6"/>
+            <mass value="1e-5" />
+            <origin xyz="0 0 0" rpy=" 0 0 0" />
+            <inertia ixx="1e-6" ixy="0" ixz="0" iyy="1e-6" iyz="0" izz="1e-6" />
         </inertial>
     </link>
-     <joint type="fixed" name="hokuyo_joint">
-        <origin xyz="0.15 0 0.1" rpy="0 0 0"/>
-        <child link="hokuyo"/>
-        <parent link="chassis"/>
-        <axis xyz="0 1 0" rpy="0 0 0"/>
+    <joint type="fixed" name="hokuyo_joint">
+        <origin xyz="0.2 0 0.1" rpy="0 0 0" />
+        <child link="hokuyo" />
+        <parent link="chassis" />
+        <axis xyz="0 1 0" rpy="0 0 0" />
     </joint>
     <gazebo reference="chassis">
-        <material>Gazebo/Blue</material>
+        <material>Gazebo/Turquoise</material>
     </gazebo>
     <gazebo reference="left_wheel">
-        <material>Gazebo/Green</material>
+        <material>Gazebo/BlueGlow</material>
     </gazebo>
     <gazebo reference="right_wheel">
-        <material>Gazebo/Green</material>
+        <material>Gazebo/BlueGlow</material>
     </gazebo>
     <gazebo reference="camera">
-        <material>Gazebo/Red</material>
+        <material>Gazebo/FlatBlack</material>
     </gazebo>
 </robot>

Commit message: Finalized the project

File: catkin_ws/src/my_robot/urdf/my_robot.xacro (robot description, xacro)
@@ -169,5 +169,5 @@
     </joint>
     <gazebo reference="chassis">
-        <material>Gazebo/Turquoise</material>
+        <material>Gazebo/PurpleGlow</material>
     </gazebo>
     <gazebo reference="left_wheel">

Commit message: Update my_robot.xacro

File: catkin_ws/src/my_robot/urdf/my_robot.xacro (robot description, xacro)
@@ -12,5 +12,5 @@
         <visual name="chassis_visual">
             <geometry>
-                <box size='0.6 0.45 0.2' />
+                <box size='0.6 0.50 0.2' />
             </geometry>
             <origin xyz="0 0 0" rpy="0 0 0" />
@@ -18,5 +18,5 @@
         <collision name="chassis_collision">
             <geometry>
-                <box size='0.6 0.3 0.2' />
+                <box size='0.6 0.50 0.2' />
             </geometry>
             <origin xyz="0 0 0" rpy="0 0 0" />
@@ -32,5 +32,5 @@
         </inertial>
         <collision name='back_caster_collision'>
-            <origin xyz="-0.15 0 -0.05" rpy=" 0 0 0" />
+            <origin xyz="-0.25 0 -0.15" rpy=" 0 0 0" />
             <geometry>
                 <sphere radius="0.0499" />
@@ -38,5 +38,5 @@
         </collision>
         <visual name='back_caster_visual'>
-            <origin xyz="-0.15 0 -0.05" rpy=" 0 0 0" />
+            <origin xyz="-0.25 0 -0.15" rpy=" 0 0 0" />
             <geometry>
                 <sphere radius="0.05" />
@@ -44,5 +44,5 @@
         </visual>
         <collision name='front_caster_collision'>
-            <origin xyz="0.15 0 -0.05" rpy=" 0 0 0" />
+            <origin xyz="0.25 0 -0.15" rpy=" 0 0 0" />
             <geometry>
                 <sphere radius="0.0499" />
@@ -50,5 +50,5 @@
         </collision>
         <visual name='front_caster_visual'>
-            <origin xyz="0.15 0 -0.05" rpy=" 0 0 0" />
+            <origin xyz="0.25 0 -0.15" rpy=" 0 0 0" />
             <geometry>
                 <sphere radius="0.05" />
@@ -60,5 +60,5 @@
             <origin xyz="0 0 0" rpy=" 0 1.5707 1.5707" />
             <geometry>
-                <cylinder radius="0.15" length="0.05" />
+                <cylinder radius="0.20" length="0.05" />
             </geometry>
         </collision>
@@ -66,5 +66,5 @@
             <origin xyz="0 0 0" rpy=" 0 1.5707 1.5707" />
             <geometry>
-                <cylinder radius="0.15" length="0.05" />
+                <cylinder radius="0.20" length="0.05" />
             </geometry>
         </visual>
@@ -83,5 +83,5 @@
             <origin xyz="0 0 0" rpy=" 0 1.5707 1.5707" />
             <geometry>
-                <cylinder radius="0.15" length="0.05" />
+                <cylinder radius="0.20" length="0.05" />
             </geometry>
         </collision>
@@ -89,5 +89,5 @@
             <origin xyz="0 0 0" rpy=" 0 1.5707 1.5707" />
             <geometry>
-                <cylinder radius="0.15" length="0.05" />
+                <cylinder radius="0.20" length="0.05" />
             </geometry>
         </visual>
